File: zigbee-raspberry-module.kicad_pcb (KiCad board)
At the start: 2 copper layers, 23.1 x 45.7 mm, 12 parts, among them J1 Conn_02x05_Odd_Even, U1 CC2538_CC2592, U2 DS3231M

Commit message: Initial commit
Parts:
- J1: moved to F.Cu
- moved J1 2.54 mm to (157.7, 110.5), turned to 270 degrees
Routing:
- net GND: track 82.9 -> 79.4 mm
- net SDA: track 37.6 -> 34.8 mm
- net SCL: track 22.1 -> 24.8 mm
- net VCC: track 98.4 -> 96.1 mm
- net RXD: track 17.1 -> 18.1 mm, vias 2 -> 1
- net TXD: track 19.4 -> 20.3 mm, vias 2 -> 1

Commit message: revision 1.1
Parts:
- removed BT1: Battery, Battery:BatteryHolder_Keystone_2998_1x6.8mm
- added J2: BK-870, BK-870:MPD_BK-870, B.Cu at (141.2, 96.0)
- J1: moved to B.Cu
- moved C1 7.37 mm to (143.3, 102.9), turned to 180 degrees
- moved R2 5.88 mm to (149.6, 89.4)
- moved R3 5.63 mm to (153.4, 89.4)
- moved R4 5.38 mm to (157.5, 89.4)
- moved RESET 5.35 mm to (148.8, 102.6), turned to 180 degrees
- moved J1 2.54 mm to (157.7, 108.0), turned to 90 degrees
- moved FLASH 0.64 mm to (155.2, 102.6), turned to 0 degrees
- moved R1 0.64 mm to (139.1, 102.9), turned to 0 degrees
- moved U2 0.43 mm to (153.2, 97.9)
Connections:
- J1 pad 1: Net-(J1-Pad1) -> VCC
- J1 pad 10: GND -> TXD
- J1 pad 2: VCC -> Net-(J1-Pad2)
- J1 pad 3: Net-(J1-Pad3) -> SDA
- J1 pad 4: SDA -> Net-(J1-Pad4)
- J1 pad 5: GND -> SCL
- J1 pad 6: SCL -> GND
- J1 pad 7: RXD -> Net-(J1-Pad7)
- J1 pad 8: Net-(J1-Pad8) -> RXD
- J1 pad 9: TXD -> GND
Routing:
- net VCC: track 96.1 -> 75.2 mm, vias 1 -> 6
- net SDA: track 34.8 -> 24.9 mm
- net RST: track 41.5 -> 51.1 mm
- net Net-(J2-Pad1): track 8.16 -> 13.7 mm
- net GND: track 79.4 -> 73.8 mm
- net PB6: track 24.6 -> 22.6 mm
- net TMS: track 15.4 -> 13.4 mm
- net TCK: track 18.5 -> 16.5 mm
- net PB7: track 21.5 -> 19.5 mm
- net Net-(R4-Pad2): track 7.75 -> 9.49 mm
- net Net-(SW1-Pad1): track 20.2 -> 19.3 mm, vias 0 -> 2
- net SCL: track 24.8 -> 24.2 mm, vias 0 -> 1
- net RXD: track 18.1 -> 17.7 mm, vias 1 -> 0
- net TXD: track 20.3 -> 20.6 mm, vias 1 -> 0

Commit message: BOM
Routing:
- net SCL: track 24.2 -> 25.9 mm

Commit message: revision 1.1
Parts:
- C1: value 100nF -> 33uF; footprint Capacitor_SMD:C_0805_2012Metric -> Capacitor_Tantalum_SMD:CP_EIA-3216-18_Kemet-A
- moved RESET 0.51 mm to (149.4, 102.6)
- moved R1 0.40 mm to (138.7, 102.7)
- moved C1 0.28 mm to (143.5, 102.7), turned to 0 degrees
Connections:
- C1 pad 1: GND -> VCC
- C1 pad 2: VCC -> GND
Routing:
- net RST: track 51.4 -> 54.9 mm
- net GND: track 73.8 -> 72.8 mm
- net VCC: track 75.2 -> 75.8 mm
