File: zigbee-raspberry-module.sch (KiCad schematic (older format))
At the start: 12 parts, among them J1 Conn_02x05_Odd_Even, SW1 FLASH, SW2 RESET, U1 CC2538_CC2592, U2 DS3231M

Commit message: revision 1.1
Parts:
- removed BT1: Battery, Battery:BatteryHolder_Keystone_2998_1x6.8mm, symbol Device:Battery
- added J2: BK-870, MPD_BK-870, symbol BK-870:BK-870
Connections:
- net +3V3: now also J1.1 (Pin_1); no longer J1.2 (Pin_2)
- net 0: now also J1.6 (Pin_6), J1.9 (Pin_9), J2.2; no longer J1.10 (Pin_10), J1.5 (Pin_5)
- net RXD: now also J1.8 (Pin_8); no longer J1.7 (Pin_7)
- net SCL: now also J1.5 (Pin_5); no longer J1.6 (Pin_6)
- net SDA: now also J1.3 (Pin_3); no longer J1.4 (Pin_4)
- net TXD: now also J1.10 (Pin_10); no longer J1.9 (Pin_9)
- net at U2.14 (VBAT): now also J2.1, J2.3
Changed lines of the file:
@@
 Comment4 ""
 $EndDescr
-Text GLabel 7150 4750 2    50   Input ~ 0
-VCC
-Wire Wire Line
-	6750 4750 7150 4750
-Text GLabel 7150 5150 2    50   Input ~ 0
+Text GLabel 5800 4750 0    50   Input ~ 0
+VCC
+Text GLabel 5800 5150 0    50   Input ~ 0
 GND
 $Comp
@@
 	1    0    0    -1
 $EndComp
-Wire Wire Line
-	6750 5150 7150 5150
-Text GLabel 5900 5150 0    50   Input ~ 0
+Text GLabel 7450 5150 2    50   Input ~ 0
 TXD
-Text GLabel 5900 5050 0    50   Input ~ 0
+Text GLabel 7450 5050 2    50   Input ~ 0
 RXD
-Text GLabel 5900 4950 0    50   Input ~ 0
-GND
-Wire Wire Line
-	6250 4950 5900 4950
-Wire Wire Line
-	6250 5050 5900 5050
-Wire Wire Line
-	6250 5150 5900 5150
+Text GLabel 7450 4950 2    50   Input ~ 0
+GND
 Text GLabel 5600 3650 2    50   Input ~ 0
 RXD
@@
 Wire Wire Line
 	6650 3650 6650 3950
-Text GLabel 7150 4850 2    50   Input ~ 0
+Text GLabel 5800 4850 0    50   Input ~ 0
 SDA
-Text GLabel 7150 4950 2    50   Input ~ 0
+Text GLabel 5800 4950 0    50   Input ~ 0
 SCL
-Wire Wire Line
-	6750 4850 7150 4850
-Wire Wire Line
-	6750 4950 7150 4950
 $Comp
 L Timer_RTC:DS3231M U2
@@
 	2300 5050 2400 5050
 $Comp
-L Device:Battery BT1
-U 1 1 5F703E18
-P 4050 5200
-F 0 "BT1" H 4158 5246 50  0000 L CNN
-F 1 "Battery" H 4158 5155 50  0000 L CNN
-F 2 "Battery:BatteryHolder_Keystone_2998_1x6.8mm" V 4050 5260 50  0001 C CNN
-F 3 "~" V 4050 5260 50  0001 C CNN
-	1    4050 5200
-	1    0    0    -1
-$EndComp
-$Comp
 L pspice:0 #GND0102
 U 1 1 5F706E26
@@
 $EndComp
 Wire Wire Line
-	4050 5400 4050 5800
-Wire Wire Line
 	3150 5650 3150 5800
 Wire Wire Line
 	3150 5800 4050 5800
-Connection ~ 4050 5800
 Wire Wire Line
 	4050 5800 4050 5950
@@
 Wire Wire Line
 	3150 4550 3150 4850
-Wire Wire Line
-	4050 4550 4050 5000
 $Comp
 L Device:R R3
@@
 	5250 2650 5800 2650
 Connection ~ 5800 2650
+$Comp
+L BK-870:BK-870 J2
+U 1 1 5FB01DD5
+P 4050 5200
+F 0 "J2" V 4004 5330 50  0000 L CNN
+F 1 "BK-870" V 4095 5330 50  0000 L CNN
+F 2 "MPD_BK-870" H 4050 5200 50  0001 L BNN
+F 3 "" H 4050 5200 50  0001 L BNN
+F 4 "MPD" H 4050 5200 50  0001 L BNN "MANUFACTURER"
+F 5 "Manufacturer Recommendation" H 4050 5200 50  0001 L BNN "STANDARD"
+F 6 "D" H 4050 5200 50  0001 L BNN "PARTREV"
+	1    4050 5200
+	0    1    1    0
+$EndComp
+Wire Wire Line
+	4050 5400 4050 5800
+Connection ~ 4050 5800
+Wire Wire Line
+	4050 4550 4050 5000
+Wire Wire Line
+	5800 4750 6250 4750
+Wire Wire Line
+	5800 4850 6250 4850
+Wire Wire Line
+	5800 4950 6250 4950
+Wire Wire Line
+	5800 5150 6250 5150
+Wire Wire Line
+	7450 5150 6750 5150
+Wire Wire Line
+	6750 5050 7450 5050
+Wire Wire Line
+	7450 4950 6750 4950
 $EndSCHEMATC

Commit message: revision 1.1
Parts:
- removed C1: 100nF, Capacitor_SMD:C_0805_2012Metric, symbol Device:C
- added C1: 33uF, Capacitor_Tantalum_SMD:CP_EIA-3216-18_Kemet-A, symbol Device:CP
Connections:
- net +3V3: now also C1.1
- net 0: now also C1.2
Changed lines of the file:
@@
 	6850 3650 6650 3650
-$Comp
-L Device:C C1
-U 1 1 5F70C06B
-P 2650 2700
-F 0 "C1" H 2765 2746 50  0000 L CNN
-F 1 "100nF" H 2765 2655 50  0000 L CNN
-F 2 "Capacitor_SMD:C_0805_2012Metric" H 2688 2550 50  0001 C CNN
-F 3 "~" H 2650 2700 50  0001 C CNN
-	1    2650 2700
-	1    0    0    -1
-$EndComp
-Wire Wire Line
-	2250 2550 2650 2550
-Connection ~ 2650 2550
-Wire Wire Line
-	2650 2550 3700 2550
 $Comp
 L power:+3.3V #PWR0101
@@
 Wire Wire Line
 	7450 4950 6750 4950
+$Comp
+L Device:CP C1
+U 1 1 5FB96F79
+P 2650 2700
+F 0 "C1" H 2532 2654 50  0000 R CNN
+F 1 "33uF" H 2532 2745 50  0000 R CNN
+F 2 "Capacitor_Tantalum_SMD:CP_EIA-3216-18_Kemet-A" H 2688 2550 50  0001 C CNN
+F 3 "~" H 2650 2700 50  0001 C CNN
+	1    2650 2700
+	-1   0    0    1
+$EndComp
+Wire Wire Line
+	2250 2550 2650 2550
+Connection ~ 2650 2550
+Wire Wire Line
+	2650 2550 3700 2550
 $EndSCHEMATC
